File: mv2_base.kicad_pcb (KiCad board)
At the start: 4 copper layers, 69 x 64 mm, 78 parts, among them J1 Conn_01x20, J2 OLED, Q1 SS8550, Q2 S8050, Q3 S8050, U1 TPS65130RGE, U3 LM5158

Commit message: Replace 500ohm resistor with 510ohm basic part
Parts:
- R16, R17, R18: value 500 -> 510
Changed lines of the file:
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@@
 			)
 		)
-		(property "Value" "500"
+		(property "Value" "510"
 			(at 0 1.17 0)
 			(layer "F.Fab")
@@
 			)
 		)
+		(property "LCSC" "C25123"
+			(at 0 0 0)
+			(unlocked yes)
+			(layer "F.Fab")
+			(hide yes)
+			(effects
+				(font
+					(size 1 1)
+					(thickness 0.15)
+				)
+			)
+		)
 		(property ki_fp_filters "R_*")
 		(sheetname "/")
@@
 			)
 		)
-		(property "Value" "500"
+		(property "Value" "510"
 			(at 0 1.17 0)
 			(layer "F.Fab")
@@
 			)
 		)
+		(property "LCSC" "C25123"
+			(at 0 0 180)
+			(unlocked yes)
+			(layer "F.Fab")
+			(hide yes)
+			(effects
+				(font
+					(size 1 1)
+					(thickness 0.15)
+				)
+			)
+		)
 		(property ki_fp_filters "R_*")
 		(sheetname "/")
@@
 			)
 		)
-		(property "Value" "500"
+		(property "Value" "510"
 			(at 0 1.17 90)
 			(layer "F.Fab")
@@
 					(thickness 0.15)
 				)
+			)
+		)
+		(property "LCSC" "C25123"
+			(at 0 0 90)
+			(unlocked yes)
+			(layer "F.Fab")
+			(hide yes)
+			(effects
+				(font
+					(size 1 1)
+					(thickness 0.15)
+				)
